File: kicad/hm-env-sensor.sch (KiCad schematic (older format))
At the start: 62 parts, among them Q1 Q12MHz/20pF/10ppm/4P/3.2x2.5mm, Q2 BC817-40(SOT23), Q3 BC817-40(SOT23), U1 BL4054B-42TPRN(SOT23-5), U2 CH340T(SSOP20W), U3 SY8089AAAC(SOT23-5), U4 BAT54C(SOT23-3), U5 ESP-WROOM-32, U6 BQ27441-G1, U7 BME280

Commit message: replace symbols and footrints by KiCAD libs + simplifiy schematic
Parts:
- removed BAT1: DW02S, OLIMEX_Connectors-FP:LIPO_BAT-CON2DW02R, symbol hm-env-sensor-rescue:BAT_CON-OLIMEX_Connectors-ESP32-DevKit-Lipo_Rev_A1-rescue
- removed C1, C6, C7: 47uF/6.3V/20%/X5R/C0805, OLIMEX_RLC-FP:C_0805_5MIL_DWS, symbol hm-env-sensor-rescue:C-OLIMEX_RCL-ESP32-DevKit-Lipo_Rev_A1-rescue
- removed C10, C11: 100nF/50V/20%/Y5V/C0603, OLIMEX_RLC-FP:C_0603_5MIL_DWS, symbol hm-env-sensor-rescue:0.1UF-25V-5%(0603)-SparkFun_BME280_Breakout_v10-eagle-impo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
- removed C2, C3: 27pF/50V/5%/C0G/C0603, OLIMEX_RLC-FP:C_0603_5MIL_DWS, symbol hm-env-sensor-rescue:C-OLIMEX_RCL-ESP32-DevKit-Lipo_Rev_A1-rescue
- removed C4: 22uF/6.3V/20%/X5R/C0603, OLIMEX_RLC-FP:C_0603_5MIL_DWS, symbol hm-env-sensor-rescue:C-OLIMEX_RCL-ESP32-DevKit-Lipo_Rev_A1-rescue
- removed C5: 100nF/50V/20%/Y5V/C0603, OLIMEX_RLC-FP:C_0603_5MIL_DWS, symbol hm-env-sensor-rescue:C-OLIMEX_RCL-ESP32-DevKit-Lipo_Rev_A1-rescue
- removed C8: 1.0uF/16V/10%/Y5V/C0603, OLIMEX_RLC-FP:C_0603_5MIL_DWS, symbol hm-env-sensor-rescue:1.0UF-16V-10%(0603)-sparkfun-battery-babysitter-eagle-impo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
- removed C9: 0.47uF/50V/20%/Y5V/C0603, OLIMEX_RLC-FP:C_0603_5MIL_DWS, symbol hm-env-sensor-rescue:CAP0603-CAP-sparkfun-battery-babysitter-eagle-import-esp32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
- removed CHARGING1: LED/YELLOW/0603, OLIMEX_LEDs-FP:LED_0603_KA, symbol hm-env-sensor-rescue:LED-OLIMEX_Diodes-ESP32-DevKit-Lipo_Rev_A1-rescue
- removed D1, D2: 1N5822/SS34/SMA, OLIMEX_Diodes-FP:SMA-KA, symbol hm-env-sensor-rescue:D_Schottky-OLIMEX_Diodes-ESP32-DevKit-Lipo_Rev_A1-rescue
- removed D_Com1, GND1: TESTPAD, OLIMEX_Other-FP:TESTPAD_40-ROUND, symbol hm-env-sensor-rescue:TESTPAD-OLIMEX_OTHER-ESP32-DevKit-Lipo_Rev_A1-rescue
- removed EXT1, EXT2: HN1x19, OLIMEX_Connectors-FP:HN1x19, symbol hm-env-sensor-rescue:CON19-OLIMEX_Connectors-ESP32-DevKit-Lipo_Rev_A1-rescue
- removed FET1: WPM2015-3/TR, OLIMEX_Transistors-FP:SOT23, symbol hm-env-sensor-rescue:P-MOS+DIOD-OLIMEX_Transistors-ESP32-DevKit-Lipo_Rev_A1-res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
- removed FID3: Fiducial, OLIMEX_Other-FP:Fiducial1x3, symbol hm-env-sensor-rescue:Fiducial-OLIMEX_OTHER-ESP32-DevKit-Lipo_Rev_A1-rescue
- removed L1: 2.2uH/1.5A/DCR<0.1R/CD32, OLIMEX_RLC-FP:CD32, symbol hm-env-sensor-rescue:L-OLIMEX_RCL-ESP32-DevKit-Lipo_Rev_A1-rescue
- removed PWRLED1: LED/RED/0603, OLIMEX_LEDs-FP:LED_0603_KA, symbol hm-env-sensor-rescue:LED-OLIMEX_Diodes-ESP32-DevKit-Lipo_Rev_A1-rescue
- removed Q1: Q12MHz/20pF/10ppm/4P/3.2x2.5mm, OLIMEX_Crystal-FP:TSX-3.2x2.5mm_GND(3), symbol hm-env-sensor-rescue:Crystal_GND-OLIMEX_Devices-ESP32-DevKit-Lipo_Rev_A1-rescue
- removed Q2, Q3: BC817-40(SOT23), OLIMEX_Transistors-FP:SOT23, symbol hm-env-sensor-rescue:Q_NPN_BEC-OLIMEX_Transistors-ESP32-DevKit-Lipo_Rev_A1-resc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
- removed R1: 10k/R0603, OLIMEX_RLC-FP:R_0603_5MIL_DWS, symbol hm-env-sensor-rescue:R-OLIMEX_RCL-ESP32-DevKit-Lipo_Rev_A1-rescue
- removed R10, R6, R7: 220R/R0603, OLIMEX_RLC-FP:R_0603_5MIL_DWS, symbol hm-env-sensor-rescue:R-OLIMEX_RCL-ESP32-DevKit-Lipo_Rev_A1-rescue
- removed R11: 4.99k/1%/R0603, OLIMEX_RLC-FP:R_0603_5MIL_DWS, symbol hm-env-sensor-rescue:R-OLIMEX_RCL-ESP32-DevKit-Lipo_Rev_A1-rescue
- removed R12: 1.1k/1%/R0603, OLIMEX_RLC-FP:R_0603_5MIL_DWS, symbol hm-env-sensor-rescue:R-OLIMEX_RCL-ESP32-DevKit-Lipo_Rev_A1-rescue
- removed R13, R8, R9: 1k/R0603, OLIMEX_RLC-FP:R_0603_5MIL_DWS, symbol hm-env-sensor-rescue:R-OLIMEX_RCL-ESP32-DevKit-Lipo_Rev_A1-rescue
- removed R14, R5: NA/R0603, OLIMEX_RLC-FP:R_0603_5MIL_DWS, symbol hm-env-sensor-rescue:R-OLIMEX_RCL-ESP32-DevKit-Lipo_Rev_A1-rescue
- removed R15: 0.01/1%/R1206, OLIMEX_RLC-FP:R_1206_5MIL_DWS, symbol hm-env-sensor-rescue:RESISTOR1206-sparkfun-battery-babysitter-eagle-import-esp3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
- removed R16, R26: 10k/R0603, OLIMEX_RLC-FP:R_0603_5MIL_DWS, symbol hm-env-sensor-rescue:4.7KOHM-1_10W-1%(0603)-SparkFun_BME280_Breakout_v10-eagle-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
- removed R17, R19, R20, R21: 4.7k/R0603, OLIMEX_RLC-FP:R_0603_5MIL_DWS, symbol hm-env-sensor-rescue:4.7KOHM-1_10W-1%(0603)-SparkFun_BME280_Breakout_v10-eagle-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
- removed R2, R3, R4: 2.2k/R0603, OLIMEX_RLC-FP:R_0603_5MIL_DWS, symbol hm-env-sensor-rescue:R-OLIMEX_RCL-ESP32-DevKit-Lipo_Rev_A1-rescue
- removed R22, R24: 330/R0603, OLIMEX_RLC-FP:R_0603_5MIL_DWS, symbol hm-env-sensor-rescue:4.7KOHM-1_10W-1%(0603)-SparkFun_BME280_Breakout_v10-eagle-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
- removed RST1, RST2, RST3: IT-1185AU2-160G-G-TR, OLIMEX_Buttons-FP:IT1185AU2_V2, symbol hm-env-sensor-rescue:SIDE_WTCM-TR(3x4)-OLIMEX_Buttons-ESP32-DevKit-Lipo_Rev_A1-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
- removed U1: BL4054B-42TPRN(SOT23-5), OLIMEX_IC-FP:SOT-23-5, symbol hm-env-sensor-rescue:BL4054B-42TPRN(SOT23-5)-OLIMEX_IC-ESP32-DevKit-Lipo_Rev_A1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
- removed U2: CH340T(SSOP20W), OLIMEX_IC-FP:SSOP-20W, symbol hm-env-sensor-rescue:CH340T(SSOP20W)-OLIMEX_IC-ESP32-DevKit-Lipo_Rev_A1-rescue
- removed U3: SY8089AAAC(SOT23-5), OLIMEX_Regulators-FP:SOT-23-5, symbol hm-env-sensor-rescue:SY8009AAAC(SOT23-5)-OLIMEX_IC-ESP32-DevKit-Lipo_Rev_A1-res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
- removed U4: BAT54C(SOT23-3), OLIMEX_Diodes-FP:SOT23-3, symbol hm-env-sensor-rescue:BAT54C(SOT23-3)-OLIMEX_Diodes-ESP32-DevKit-Lipo_Rev_A1-res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
- removed U5: ESP-WROOM-32, OLIMEX_Cases-FP:ESP-WROOM-32_MODULE, symbol hm-env-sensor-rescue:ESP-WROOM-32-OLIMEX_Cases-ESP32-DevKit-Lipo_Rev_A1-rescue
- removed U6: BQ27441-G1, sparkfun-battery-babysitter:PDSO-N12, symbol hm-env-sensor-rescue:BQ27441-G1-sparkfun-battery-babysitter-eagle-import-esp32-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
- removed U7: BME280, SparkFun_BME280_Breakout_v10:BME280_LGA, symbol hm-env-sensor-rescue:BME280-SparkFun_BME280_Breakout_v10-eagle-import-ESP32-Dev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
- removed USB-UART1: MISB-SWMM-5B-LF(USB_MICRO), OLIMEX_Connectors-FP:USB-MICRO_MISB-SWMM-5B_LF, symbol hm-env-sensor-rescue:USB-MINI-OLIMEX_Connectors-ESP32-DevKit-Lipo_Rev_A1-rescue
- added BAT1: Conn_01x02_Male, Connector_Wuerth:Wuerth_WR-WTB_64800211622_1x02_P1.50mm_Vertical, symbol Connector:Conn_01x02_Male
- added C1: 47u/6.3V, Capacitor_SMD:C_0805_2012Metric_Pad1.15x1.40mm_HandSolder, symbol Device:C
- added C10, C11, C5: 100n/50V, Capacitor_SMD:C_0603_1608Metric_Pad1.05x0.95mm_HandSolder, symbol Device:C
- added C12: 100p/6.3V, Capacitor_SMD:C_0805_2012Metric_Pad1.15x1.40mm_HandSolder, symbol Device:C
- added C2, C3: 27p/50V/C0G, Capacitor_SMD:C_0603_1608Metric_Pad1.05x0.95mm_HandSolder, symbol Device:C
- added C4: 22u/6.3V, Capacitor_SMD:C_0603_1608Metric_Pad1.05x0.95mm_HandSolder, symbol Device:C
- added C6, C7: 10u/6.3V, Capacitor_SMD:C_0805_2012Metric_Pad1.15x1.40mm_HandSolder, symbol Device:C
- added C8: 1u/16V, Capacitor_SMD:C_0603_1608Metric_Pad1.05x0.95mm_HandSolder, symbol Device:C
- added C9: 470n/50V, Capacitor_SMD:C_0603_1608Metric_Pad1.05x0.95mm_HandSolder, symbol Device:C
- added CHARGING1: LED/Yellow, LED_SMD:LED_0603_1608Metric_Pad1.05x0.95mm_HandSolder, symbol Device:LED
- added D1, D2: 1N5822, Diode_SMD:D_SMC_Handsoldering, symbol Diode:1N5822
- added D?: BAT54C, Package_TO_SOT_SMD:SOT-23, symbol Diode:BAT54C
- added FET1: WPM2015-3/TR, symbol Device:Q_PMOS_GSD
- added FID1: Fiducial, symbol Mechanical:Fiducial
- added FID2, FID3: Fiducial, Fiducial:Fiducial_1mm_Mask2mm, symbol Mechanical:Fiducial
- added J1: USB_B_Micro, Connector_USB:USB_Micro-B_Molex_47346-0001, symbol Connector:USB_B_Micro
- added L1: 4.7uH/1.4A/DCR<0.1R/CD32, symbol Device:L
- added PWRLED1: LED/Red, LED_SMD:LED_0603_1608Metric_Pad1.05x0.95mm_HandSolder, symbol Device:LED
- added Q1: Q12MHz/20pF/10ppm/4P, Crystal:Crystal_SMD_TXC_7M-4Pin_3.2x2.5mm_HandSoldering, symbol Device:Crystal_GND2_Small
- added Q2, Q3: BC817, Package_TO_SOT_SMD:SOT-23, symbol Transistor_BJT:BC817
- added R1, R16, R2, R26: 10k, Resistor_SMD:R_0603_1608Metric_Pad1.05x0.95mm_HandSolder, symbol Device:R
- added R10, R6, R7: 220, Resistor_SMD:R_0603_1608Metric_Pad1.05x0.95mm_HandSolder, symbol Device:R
- added R11: 540k, Resistor_SMD:R_0603_1608Metric_Pad1.05x0.95mm_HandSolder, symbol Device:R
- added R12: 120k, Resistor_SMD:R_0603_1608Metric_Pad1.05x0.95mm_HandSolder, symbol Device:R
- added R13, R8, R9: 1k, Resistor_SMD:R_0603_1608Metric_Pad1.05x0.95mm_HandSolder, symbol Device:R
- added R14, R5: NA, Resistor_SMD:R_0603_1608Metric_Pad1.05x0.95mm_HandSolder, symbol Device:R
- added R15: 0.01/1%, Resistor_SMD:R_1206_3216Metric_Pad1.42x1.75mm_HandSolder, symbol Device:R
- added R17, R19, R20, R21: 4.7k, Resistor_SMD:R_0603_1608Metric_Pad1.05x0.95mm_HandSolder, symbol Device:R
- added R18, R24: 330, Resistor_SMD:R_0603_1608Metric_Pad1.05x0.95mm_HandSolder, symbol Device:R
- added R3, R4: 2.2k, Resistor_SMD:R_0603_1608Metric_Pad1.05x0.95mm_HandSolder, symbol Device:R
- added RST2, RST3: SW_Push, Button_Switch_SMD:SW_Push_1P1T_NO_CK_KSC6xxJ, symbol Switch:SW_Push
- added TP?: D_Com1, TestPoint:TestPoint_THTPad_D2.0mm_Drill1.0mm, symbol Connector:TestPoint
- added TP?: GND, TestPoint:TestPoint_THTPad_D2.0mm_Drill1.0mm, symbol Connector:TestPoint
- added TP?: 5V, TestPoint:TestPoint_THTPad_D2.0mm_Drill1.0mm, symbol Connector:TestPoint
- added TP?: 3.3V, TestPoint:TestPoint_THTPad_D2.0mm_Drill1.0mm, symbol Connector:TestPoint
- added U1: LTC4054ES5-4.2, Package_TO_SOT_SMD:TSOT-23-5, symbol Battery_Management:LTC4054ES5-4.2
- added U2: CH340T, Package_SO:SSOP-20_5.3x7.2mm_P0.65mm, symbol Interface_USB:CH340T
- added U3: PAM2305AABADJ, Package_TO_SOT_SMD:TSOT-23-5, symbol Regulator_Switching:PAM2305AABADJ
- added U5: ESP32-WROOM-32, RF_Module:ESP32-WROOM-32, symbol RF_Module:ESP32-WROOM-32
- added U6: BQ27441-G1, Package_SON:Texas_S-PDSO-N12, symbol Battery_Management:BQ27441-G1
- added U7: BME280, Package_LGA:Bosch_LGA-8_2.5x2.5mm_P0.65mm_ClockwisePinNumbering, symbol Sensor:BME280
- D4: value LED/GREEN/0603 -> LED/Green; footprint OLIMEX_LEDs-FP:LED_0603_KA -> LED_SMD:LED_0603_1608Metric_Pad1.05x0.95mm_HandSolder
- D6: value LED/RED/0603 -> LED/Green; footprint OLIMEX_LEDs-FP:LED_0603_KA -> LED_SMD:LED_0603_1608Metric_Pad1.05x0.95mm_HandSolder
Connections:
- net labels added: SCL, SDA
- net labels removed: 3.3V, GPIO26, GPIO27
- wire segments 305 -> 241
- no-connect marks 6 -> 7
Other:
- note added: "GPIO2 must also be either left unconnected/floating, \nor driven Low, in order to enter the serial bootloader."
- note added: "The ESP32 will enter the serial bootloader \nwhen GPIO0 is held low on reset. \nOtherwise it will run the program in flash."
- note removed: "ESP-WROOM-32 MODULE"
- note removed: "Extensions"
- note removed: "Two reset button, we keep the original \nplacement of the reset button, and \nwe add a reset button that will be \naccessible via the ventilation holes in the enclosure."

Commit message: aktuell
Parts:
- removed FET1: WPM2015-3/TR, symbol Device:Q_PMOS_GSD
- removed J1: USB_B_Micro, Connector_USB:USB_Micro-B_Molex_47346-0001, symbol Connector:USB_B_Micro
- removed Q1: Q12MHz/20pF/10ppm/4P, Crystal:Crystal_SMD_TXC_7M-4Pin_3.2x2.5mm_HandSoldering, symbol Device:Crystal_GND2_Small
- added H1, H2, H3, H4: MountingHole, MountingHole:MountingHole_3.2mm_M3, symbol Mechanical:MountingHole
- added J2: Conn_01x06_Female, Connector_PinSocket_2.54mm:PinSocket_1x06_P2.54mm_Vertical, symbol Connector:Conn_01x06_Female
- added P?: USB_C_Plug_USB2.0, Connector_USB:USB_C_Receptacle_Amphenol_12401548E4-2A, symbol Connector:USB_C_Plug_USB2.0
- added Q4: NTR4101PT1G, Package_TO_SOT_SMD:SOT-23, symbol Device:Q_PMOS_GSD
- added R22, R27: 10k, Resistor_SMD:R_0603_1608Metric_Pad1.05x0.95mm_HandSolder, symbol Device:R
- added R23, R25: dnp, Resistor_SMD:R_0603_1608Metric_Pad1.05x0.95mm_HandSolder, symbol Device:R
- added Y1: 12 MHz, Crystal:Crystal_SMD_HC49-SD_HandSoldering, symbol Device:Crystal
- BAT1: footprint Connector_Wuerth:Wuerth_WR-WTB_64800211622_1x02_P1.50mm_Vertical -> Connector_JST:JST_PH_S2B-PH-K_1x02_P2.00mm_Horizontal; Part Nr. (none) -> JST PH2P ST90; Supplier (none) -> Reichelt
- C2, C3: value 27p/50V/C0G -> 22p/50V/C0G
- D6: value LED/Green -> LED/Blue
- FID1: footprint (none) -> Fiducial:Fiducial_1mm_Mask2mm
- L1: value 4.7uH/1.4A/DCR<0.1R/CD32 -> 4.7u; footprint (none) -> Inductor_SMD:L_Wuerth_WE-TPC-3816; Part Nr. (none) -> WUE 744031004; Supplier (none) -> Reichelt
- RST2, RST3: footprint Button_Switch_SMD:SW_Push_1P1T_NO_CK_KSC6xxJ -> Button_Switch_SMD:SW_SPST_PTS645; Supplier (none) -> lab
- gave numbers to parts that had none: 5
Connections:
- net labels added: BAT_LOW, USER_LED_Blue, USER_LED_Green
- net labels removed: GPI34, GPI35, GPI36/SENSOR_VP, GPI39/SENSOR_VN, GPIO10/SD_DATA3, GPIO11/SD_CMD, GPIO12, GPIO14, GPIO15, GPIO16, GPIO17, GPIO18, GPIO19, GPIO21, GPIO22, GPIO23, GPIO25, GPIO32, GPIO33, GPIO4, GPIO5, GPIO6/SD_CLK, GPIO7/SD_DATA0, GPIO8/SD_DATA1, GPIO9/SD_DATA2
- wire segments 241 -> 256
- no-connect marks 7 -> 12
Other:
- note added: "1.5 MHz"
- note added: "BMExxx breakout board or BMExxx Chip direct"
- note added: "Connector for \nBME280/BME680\nBreakout boards\n5: CS/SDO\n6: SDO/CS\n"
- note added: "Connector: Reichelt - JST PH2P BU\nCrimp: JST PH CKB"
- note added: "Mounting Holes:"
- note removed: "Application LEDs"
- note removed: "BME280"
- note removed: "PENDING"
- moved on the sheet: BAT1, C10, C11, C6, C9, D4, D6, FID1, FID2, FID3, R13, R14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
